File: LEDpanel.kicad_sch (KiCad schematic)
At the start: 56 parts, among them J1 Barrel_Jack_Switch, J2 Barrel_Jack_Switch, J3 Conn_01x02, J4 TESTPOINTS, Q1 MJE31D, Q2 MJE31D, Q3 MJE31D, SW1 SW_SPST, U1 LM358, U2 LM358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

Commit message: Send to JLCPCB
Parts:
- D2, D3, D4: LCSC C2099 -> C81598
Changed lines of the file:
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@@
       (effects (font (size 1.27 1.27)) hide)
     )
-    (property "LCSC" "C2099" (at 66.675 60.325 90)
+    (property "LCSC" "C81598" (at 66.675 60.325 90)
       (effects (font (size 1.27 1.27)) hide)
     )
@@
       (effects (font (size 1.27 1.27)) hide)
     )
-    (property "LCSC" "C2099" (at 66.675 68.58 90)
+    (property "LCSC" "C81598" (at 66.675 68.58 90)
       (effects (font (size 1.27 1.27)) hide)
     )
@@
       (effects (font (size 1.27 1.27)) hide)
     )
-    (property "LCSC" "C2099" (at 66.675 51.435 90)
-      (effects (font (size 1.27 1.27)) hide)
-    )
+    (property "LCSC" "C81598" (at 66.675 51.435 90)
+      (effects (font (size 1.27 1.27)) hide)
+    )
